File: pixxy-kicad/pixxy.kicad_pcb (KiCad board)
At the start: 2 copper layers, 55.5 x 98 mm, 24 parts, among them Q1 2N3904, SW17 SW_SPDT, U1 Pico

Commit message: Add initial working software, improve PCB design
Connections:
- RV1 pad 1: GND -> +3.3V
- RV1 pad 3: +3.3V -> GND
- RV2 pad 1: GND -> +3.3V
- RV2 pad 3: +3.3V -> GND
- RV3 pad 1: GND -> +3.3V
- RV3 pad 3: +3.3V -> GND
- U1 pad 38: GND -> unconnected-(U1-GND-Pad38)
Routing:
- net GND: track 78.5 -> 36.4 mm, vias 1 -> 0
- net +3.3V: track 92.6 -> 80.1 mm
Other:
- board text added: "Effect 3"
- board text added: "Select one of the preset colours by clicking on the oolour buttons, or mix using the RGB pots. After selecting a colour, you can send it using the fade/flash button. You can make these commands repeat by turning the switch below these buttons to 'Repeat'. You can change the speed by holding down the 'Speed' button and turning the 'Blue' potentiometer. If you have a X2 (Taylor) bracelet, you can u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"
- board text added: "Taylor reset"
- board text removed: "Select a colour or use a custom one by using the RGB pots and the custom button. Send the colour using the fade/flash button. Repeat these commands by turning the switch to 'Repeat'. Speed can be changed by holding down the Speed Set button whilst turning the 'Blue' knob. On/Off button and Rainbow/Taylor End effects only work on X2 (Taylor) bracelets."
- board text removed: "Speed Set"
- board text removed: "Taylor End"

Commit message: Add rev1 pcb files
Parts:
- R1: value 15R -> 10R
Connections:
- net Net-(Q1-B) renamed /LED_SIG
- net Net-(SW17-A) renamed /SW_ONCE_REPEAT
- net Net-(U1-GPIO10) renamed /MTX_COL4
- net Net-(U1-GPIO11) renamed /MTX_COL3
- net Net-(U1-GPIO12) renamed /MTX_COL2
- net Net-(U1-GPIO13) renamed /MTX_COL1
- net Net-(U1-GPIO26_ADC0) renamed /POT_R
- net Net-(U1-GPIO27_ADC1) renamed /POT_G
- net Net-(U1-GPIO28_ADC2) renamed /POT_B
- net Net-(U1-GPIO6) renamed /MTX_ROW4
- net Net-(U1-GPIO7) renamed /MTX_ROW3
- net Net-(U1-GPIO8) renamed /MTX_ROW2
- net Net-(U1-GPIO9) renamed /MTX_ROW1
- RV1 pad 1: +3.3V -> GND
- RV1 pad 3: GND -> +3.3V
- RV2 pad 1: +3.3V -> GND
- RV2 pad 3: GND -> +3.3V
- RV3 pad 1: +3.3V -> GND
- RV3 pad 3: GND -> +3.3V
- U1 pad 38: unconnected-(U1-GND-Pad38) -> GND
Routing:
- net GND: track 36.4 -> 78.5 mm, vias 0 -> 1
- net +3.3V: track 80.1 -> 92.6 mm
Other:
- board text added: "Select a colour or use a custom one by using the RGB pots and the custom button. Send the colour using the fade/flash button. Repeat these commands by turning the switch to 'Repeat'. Speed can be changed by holding down the Speed Set button whilst turning the 'Blue' knob. On/Off button and Rainbow/Taylor End effects only work on X2 (Taylor) bracelets."
- board text added: "Speed Set"
- board text added: "Taylor End"
- board text removed: "Effect 3"
- board text removed: "Select one of the preset colours by clicking on the oolour buttons, or mix using the RGB pots. After selecting a colour, you can send it using the fade/flash button. You can make these commands repeat by turning the switch below these buttons to 'Repeat'. You can change the speed by holding down the 'Speed' button and turning the 'Blue' potentiometer. If you have a X2 (Taylor) bracelet, you can u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"
- board text removed: "Taylor reset"

Commit message: Improved schematic and finished pcb for rev2
Parts:
- added C1: 10u, Capacitor_SMD:C_0805_2012Metric, B.Cu at (47.7, 46.5)
- added C10: 100n, Capacitor_SMD:C_0402_1005Metric, B.Cu at (61.9, 57.0)
- added C11: 100n, Capacitor_SMD:C_0402_1005Metric, B.Cu at (64.4, 61.3)
- added C12: 100n, Capacitor_SMD:C_0402_1005Metric, B.Cu at (72.6, 55.6)
- added C13: 100n, Capacitor_SMD:C_0402_1005Metric, B.Cu at (74.5, 52.1)
- added C14: 15p, Capacitor_SMD:C_0402_1005Metric, B.Cu at (69.8, 62.2)
- added C15: 15p, Capacitor_SMD:C_0402_1005Metric, B.Cu at (65.1, 64.2)
- added C16: 10u, Capacitor_SMD:C_0805_2012Metric, B.Cu at (54.0, 56.8)
- added C17: 10u, Capacitor_SMD:C_0805_2012Metric, B.Cu at (82.6, 47.8)
- added C2: 100n, Capacitor_SMD:C_0402_1005Metric, B.Cu at (71.1, 42.5)
- added C3: 1u, Capacitor_SMD:C_0402_1005Metric, B.Cu at (62.0, 48.6)
- added C4: 100n, Capacitor_SMD:C_0402_1005Metric, B.Cu at (68.6, 45.9)
- added C5: 100n, Capacitor_SMD:C_0402_1005Metric, B.Cu at (64.4, 60.3)
- added C6: 1u, Capacitor_SMD:C_0402_1005Metric, B.Cu at (62.0, 49.8)
- added C7: 100n, Capacitor_SMD:C_0402_1005Metric, B.Cu at (67.5, 45.4)
- added C8: 100n, Capacitor_SMD:C_0402_1005Metric, B.Cu at (60.2, 51.8)
- added C9: 100n, Capacitor_SMD:C_0402_1005Metric, B.Cu at (60.2, 52.9)
- added H1: ToolingHole, MountingHole:MountingHole_1.152mm, F.Cu at (94.2, 129.2)
- added H2: ToolingHole, MountingHole:MountingHole_1.152mm, F.Cu at (43.2, 37.5)
- added J1: USB_C_Receptacle_USB2.0_14P, Connector_USB:USB_C_Receptacle_G-Switch_GT-USB-7010ASV, B.Cu at (52.0, 40.1)
- added J2: Conn_01x03, Connector_JST:JST_SH_SM03B-SRSS-TB_1x03-1MP_P1.00mm_Horizontal, B.Cu at (44.4, 59.6)
- added R2: 1k, Resistor_SMD:R_0402_1005Metric, B.Cu at (78.4, 42.2)
- added R3: 5k1, Resistor_SMD:R_0402_1005Metric, B.Cu at (59.1, 44.0)
- added R4: 27.4, Resistor_SMD:R_0402_1005Metric, B.Cu at (66.2, 48.5)
- added R5: 27.4, Resistor_SMD:R_0402_1005Metric, B.Cu at (65.2, 48.5)
- added R6: DNF, Resistor_SMD:R_0402_1005Metric, B.Cu at (81.2, 44.6)
- added R7: 5k1, Resistor_SMD:R_0402_1005Metric, B.Cu at (50.5, 47.0)
- added R8: 1k, Resistor_SMD:R_0402_1005Metric, B.Cu at (66.8, 62.2)
- added TP1: TestPoint, TestPoint:TestPoint_Pad_1.5x1.5mm, B.Cu at (82.2, 42.2)
- added U2: W25Q128JVS, Package_SO:SOIC-8_5.23x5.23mm_P1.27mm, B.Cu at (74.2, 46.5)
- added U3: NCP1117-3.3_SOT223, Package_TO_SOT_SMD:SOT-223-3_TabPin2, B.Cu at (51.8, 52.0)
- added Y1: ABM8-272-T3, Crystal:Crystal_SMD_3225-4Pin_3.2x2.5mm, B.Cu at (68.1, 65.0)
- U1: value Pico -> RP2040; footprint MCU_RaspberryPi_and_Boards:RPi_Pico_SMD -> Package_DFN_QFN:QFN-56-1EP_7x7mm_P0.4mm_EP3.2x3.2mm
- moved SW13 52.1 mm to (84.9, 86.2)
- moved SW4 52.1 mm to (47.2, 122.2)
- moved SW14 36.3 mm to (84.9, 96.4)
- moved SW8 36.3 mm to (59.4, 122.2)
- moved SW3 31.7 mm to (47.2, 106.8)
- moved SW9 31.7 mm to (71.4, 86.2)
- moved SW12 16.8 mm to (71.4, 122.2)
- moved SW15 16.8 mm to (84.9, 112.2)
- moved SW2 16.1 mm to (47.2, 96.8)
- moved SW5 16.1 mm to (59.4, 86.2)
- moved SW10 15.6 mm to (71.4, 96.8)
- moved SW7 15.6 mm to (59.4, 106.8)
- moved Q1 8.67 mm to (60.7, 39.0)
- moved D1 5.22 mm to (67.9, 39.0)
- moved R1 3.44 mm to (85.5, 39.0)
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Connections:
- R1 pad 1: +3.3V -> +3V3
- RV1 pad 3: +3.3V -> +3V3
- RV2 pad 3: +3.3V -> +3V3
- RV3 pad 3: +3.3V -> +3V3
- SW10 pad 1: /MTX_COL2 -> /MTX_COL3
- SW10 pad 2: /MTX_ROW3 -> /MTX_ROW2
- SW12 pad 1: /MTX_COL4 -> /MTX_COL3
- SW12 pad 2: /MTX_ROW3 -> /MTX_ROW4
- SW13 pad 1: /MTX_COL1 -> /MTX_COL4
- SW13 pad 2: /MTX_ROW4 -> /MTX_ROW1
- SW14 pad 1: /MTX_COL2 -> /MTX_COL4
- SW14 pad 2: /MTX_ROW4 -> /MTX_ROW2
- SW15 pad 1: /MTX_COL3 -> /MTX_COL4
- SW15 pad 2: /MTX_ROW4 -> /MTX_ROW3
- SW2 pad 1: /MTX_COL2 -> /MTX_COL1
- SW2 pad 2: /MTX_ROW1 -> /MTX_ROW2
- SW3 pad 1: /MTX_COL3 -> /MTX_COL1
- SW3 pad 2: /MTX_ROW1 -> /MTX_ROW3
- SW4 pad 1: /MTX_COL4 -> /MTX_COL1
- SW4 pad 2: /MTX_ROW1 -> /MTX_ROW4
- SW5 pad 1: /MTX_COL1 -> /MTX_COL2
- SW5 pad 2: /MTX_ROW2 -> /MTX_ROW1
- SW7 pad 1: /MTX_COL3 -> /MTX_COL2
- SW7 pad 2: /MTX_ROW2 -> /MTX_ROW3
- SW8 pad 1: /MTX_COL4 -> /MTX_COL2
- SW8 pad 2: /MTX_ROW2 -> /MTX_ROW4
- SW9 pad 1: /MTX_COL1 -> /MTX_COL3
- SW9 pad 2: /MTX_ROW3 -> /MTX_ROW1
- U1 pad 1: unconnected-(U1-GPIO0-Pad1) -> +3V3
- U1 pad 10: /MTX_ROW3 -> +3V3
- U1 pad 13: unconnected-(U1-GND-Pad13) -> /MTX_COL4
- U1 pad 14: /MTX_COL4 -> /MTX_COL3
- U1 pad 15: /MTX_COL3 -> /MTX_COL2
- U1 pad 16: /MTX_COL2 -> /MTX_COL1
- U1 pad 17: /MTX_COL1 -> unconnected-(U1-GPIO14-Pad17)
- U1 pad 19: unconnected-(U1-GPIO14-Pad19) -> GND
- U1 pad 20: unconnected-(U1-GPIO15-Pad20) -> /XIN
- U1 pad 21: /LED_SIG -> /XOUT
- U1 pad 22: unconnected-(U1-GPIO17-Pad22) -> +3V3
- U1 pad 23: unconnected-(U1-GND-Pad23) -> +1V1
- U1 pad 24: unconnected-(U1-GPIO18-Pad24) -> /SWCLK
- U1 pad 25: unconnected-(U1-GPIO19-Pad25) -> /SWDIO
- U1 pad 27: unconnected-(U1-GPIO21-Pad27) -> /LED_SIG
- U1 pad 31: /POT_R -> unconnected-(U1-GPIO20-Pad31)
- U1 pad 32: /POT_G -> unconnected-(U1-GPIO21-Pad32)
- U1 pad 33: unconnected-(U1-AGND-Pad33) -> +3V3
- U1 pad 34: /POT_B -> unconnected-(U1-GPIO22-Pad34)
- U1 pad 36: +3.3V -> unconnected-(U1-GPIO24-Pad36)
- U1 pad 38: GND -> /POT_R
- U1 pad 39: unconnected-(U1-VSYS-Pad39) -> /POT_G
- U1 pad 40: unconnected-(U1-VBUS-Pad40) -> /POT_B
- U1 pad 42: unconnected-(U1-GND-Pad42) -> +3V3
- U1 pad 43: unconnected-(U1-SWDIO-Pad43) -> +3V3
- U1 pad 8: unconnected-(U1-GND-Pad8) -> /MTX_ROW4
- U1 pad 9: /MTX_ROW4 -> /MTX_ROW3
Routing:
- net +3.3V: track 92.6 -> 0.00 mm
- net +3V3: track 0.00 -> 44.6 mm, vias 0 -> 2
- net GND: track 78.5 -> 44.4 mm, vias 1 -> 21
- net +1V1: track 0.00 -> 24.4 mm
- net /QSPI_SS: track 0.00 -> 22.2 mm
- net /SWCLK: track 0.00 -> 21.3 mm
- net /SWDIO: track 0.00 -> 20.4 mm
- net /USB_D-: track 0.00 -> 19.5 mm
- net /USB_D+: track 0.00 -> 18.5 mm
- net /QSPI_SD1: track 0.00 -> 15.5 mm
- net VBUS: track 0.00 -> 12.9 mm
- net /POT_B: track 34.4 -> 46.9 mm, vias 0 -> 1
- net /POT_R: track 41.1 -> 28.9 mm, vias 0 -> 1
- net /QSPI_SD2: track 0.00 -> 11.0 mm
- net /XIN: track 0.00 -> 9.34 mm
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- added copper zone on B.Cu, net +3V3
- added copper zone on B.Cu, net GND
Other:
- board size 55.5 x 98 mm -> 55.5 x 96.2 mm
- board text added: "Select a colour or use a custom one by using the custom button and the R/G/B pots. Send the colour with the fade or flash button. Repeat these commands by setting the switch to Repeat. Speed can be changed by holding down the Speed Set button whilst turning the Blue knob. On/Off button and Rainbow/Taylor End effects only work on X2 (Taylor) bracelets."
- board text added: "Short to GND for BOOTSEL"
- board text added: "© Wouter de Droog - rev. 2 (210924)"
- board text removed: "Select a colour or use a custom one by using the RGB pots and the custom button. Send the colour using the fade/flash button. Repeat these commands by turning the switch to 'Repeat'. Speed can be changed by holding down the Speed Set button whilst turning the 'Blue' knob. On/Off button and Rainbow/Taylor End effects only work on X2 (Taylor) bracelets."
- board text removed: "© Wouter de Droog - rev. 1 (210824)"
